File: Gruppo4SensoriIR/Gruppo4SensoriIR.kicad_sch (KiCad schematic)
At the start: 30 parts, among them J1 Conn_01x06_Male, U1 Opamp_Quad

Commit message: Add files via upload
Parts:
- U1: value Opamp_Quad -> LM124-LM324
- U1: value Opamp_Quad -> LM124-LM324; footprint Package_DIP:DIP-14_W7.62mm_LongPads -> (none)
Changed lines of the file:
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@@
     (in_bom yes) (on_board yes) (fields_autoplaced)
     (property "Reference" "U1" (id 0) (at 127 48.26 0))
-    (property "Value" "Opamp_Quad" (id 1) (at 127 50.8 0))
+    (property "Value" "LM124-LM324" (id 1) (at 127 50.8 0))
     (property "Footprint" "" (id 2) (at 127 58.42 0)
       (effects (font (size 1.27 1.27)) hide)
@@
     (in_bom yes) (on_board yes) (fields_autoplaced)
     (property "Reference" "U1" (id 0) (at 76.2 48.26 0))
-    (property "Value" "Opamp_Quad" (id 1) (at 76.2 50.8 0))
+    (property "Value" "LM124-LM324" (id 1) (at 76.2 50.8 0))
     (property "Footprint" "" (id 2) (at 76.2 58.42 0)
       (effects (font (size 1.27 1.27)) hide)
@@
     (in_bom yes) (on_board yes) (fields_autoplaced)
     (property "Reference" "U1" (id 0) (at 151.13 48.26 0))
-    (property "Value" "Opamp_Quad" (id 1) (at 151.13 50.8 0))
-    (property "Footprint" "Package_DIP:DIP-14_W7.62mm_LongPads" (id 2) (at 151.13 58.42 0)
+    (property "Value" "LM124-LM324" (id 1) (at 151.13 50.8 0))
+    (property "Footprint" "" (id 2) (at 151.13 58.42 0)
       (effects (font (size 1.27 1.27)) hide)
     )
@@
       (effects (font (size 1.27 1.27)) (justify left))
     )
-    (property "Value" "Opamp_Quad" (id 1) (at 172.72 59.6899 0)
+    (property "Value" "LM124-LM324" (id 1) (at 172.72 59.6899 0)
       (effects (font (size 1.27 1.27)) (justify left))
     )
@@
     (in_bom yes) (on_board yes) (fields_autoplaced)
     (property "Reference" "U1" (id 0) (at 101.6 48.26 0))
-    (property "Value" "Opamp_Quad" (id 1) (at 101.6 50.8 0))
+    (property "Value" "LM124-LM324" (id 1) (at 101.6 50.8 0))
     (property "Footprint" "" (id 2) (at 101.6 58.42 0)
       (effects (font (size 1.27 1.27)) hide)
@@
     )
     (path "/2e0a078d-e198-4697-954d-d9db9f38dbb4"
-      (reference "U1") (unit 1) (value "Opamp_Quad") (footprint "")
+      (reference "U1") (unit 1) (value "LM124-LM324") (footprint "")
     )
     (path "/b0cc25b3-a5e9-4f32-be8e-2d0b44b84572"
-      (reference "U1") (unit 2) (value "Opamp_Quad") (footprint "")
+      (reference "U1") (unit 2) (value "LM124-LM324") (footprint "")
     )
     (path "/11fe33d5-ff33-4858-a950-602bb22d88aa"
-      (reference "U1") (unit 3) (value "Opamp_Quad") (footprint "")
+      (reference "U1") (unit 3) (value "LM124-LM324") (footprint "")
     )
     (path "/4d7494e5-88b7-400a-9ab6-eb9787a9bce3"
-      (reference "U1") (unit 4) (value "Opamp_Quad") (footprint "Package_DIP:DIP-14_W7.62mm_LongPads")
+      (reference "U1") (unit 4) (value "LM124-LM324") (footprint "")
     )
     (path "/4f6e0209-bbef-4339-b133-c0379fef90df"
-      (reference "U1") (unit 5) (value "Opamp_Quad") (footprint "")
-    )
-  )
+      (reference "U1") (unit 5) (value "LM124-LM324") (footprint "")
+    )
+  )
